Commit message: Working on tag-driven clock

File: com_3d/urdf/irb120_with_finger.xacro (robot description, xacro)
@@ -6,31 +6,38 @@
   <xacro:include filename="$(find abb_irb120_support)/urdf/irb120_3_58.xacro"/>
   <!-- ====== Params you can tweak ====== -->
-  <xacro:property name="tool_mass" value="0.255"/>          <!-- kg (sensor+finger) (from spec sheet) -->
-  <xacro:property name="tool_cog_z" value="0.017"/>         <!-- m in tool frame (from spec sheet)-->
-  <xacro:property name="ft_z" value="0.083"/>              <!-- FT sensor height -->
-  <xacro:property name="finger_z" value="0.1143"/>          <!-- finger length (from onshape)-->
-  <!-- Total offset from link_6 to finger tip will be ft_z + finger_z -->
+  <xacro:property name="ft_mass" value="0.255"/>          <!-- kg (sensor) (from spec sheet) -->
+  <xacro:property name="ft_cog_z" value="0.063"/>         <!-- meters in tool frame (from spec sheet)-->
+  <xacro:property name="ft_length" value="0.03"/>         <!-- FT sensor length -->
+  <xacro:property name="finger_mass" value="0.066"/>      <!-- kg (finger) (from onshape) -->
+  <xacro:property name="finger_length" value="0.1143"/>   <!-- finger length (from onshape)-->
+  <!-- Total offset from link_6 to finger tip will be ft_length + finger_length -->
   <!-- ====== FT sensor link mounted to link_6 ====== -->
   <link name="ft_link">
     <inertial>
-      <origin xyz="0 0 ${tool_cog_z}" rpy="0 0 0"/>
-      <mass value="${tool_mass}"/>
-      <!-- simple diagonal inertia; refine if you have CAD -->
+      <origin xyz="0 0 ${ft_cog_z}" rpy="0 0 0"/>
+      <mass value="${ft_mass}"/>
       <inertia ixx="5e-4" iyy="5e-4" izz="5e-4" ixy="0" ixz="0" iyz="0"/>
     </inertial>
     <visual>
-      <origin xyz="0 0 ${ft_z/2}" rpy="0 0 0"/>
+      <origin xyz="0 0 ${ft_length/2}" rpy="0 0 0"/>
       <geometry>
-        <cylinder radius="0.03" length="${ft_z}"/>
+        <cylinder radius="0.025" length="${ft_length}"/>
       </geometry>
       <material name="Grey">
-        <color rgba="0.8 0.8 0.8 1.0"/>
+        <color rgba="0.6 0.6 0.6 1.0"/>
       </material>
     </visual>
+    <!-- Basic cylinder collision geom -->
+    <collision>
+        <origin xyz="0 0 ${ft_length / 4}" rpy="0 0 0"/>
+        <geometry>
+            <cylinder radius="0.025" length="${ft_length / 2}"/>
+        </geometry>
+    </collision>
   </link>
   <joint name="link_6_to_ft" type="fixed">
     <parent link="link_6"/>
     <!-- Adjust xyz/rpy to match your real mounting orientation -->
-    <origin xyz="0 0 0" rpy="0 1.5708 0"/>
+    <origin xyz="0.001 0 0" rpy="0 1.5708 0"/>
     <child link="ft_link"/>
   </joint>
@@ -40,5 +47,5 @@
     <inertial>
         <origin xyz="0 0 0.026" rpy="0 0 0"/>   <!-- adjust CoG -->
-        <mass value="0.066"/>                   <!-- kg -->
+        <mass value="${finger_mass}"/>                   <!-- kg -->
         <inertia ixx="70.297" iyy="70.297" izz="70.297" ixy="0" ixz="0" iyz="0"/> <!-- kg mm^2-->
     </inertial>
@@ -53,8 +60,15 @@
         </material>
     </visual>
+    <!-- Simple cylinder geom -->
+    <collision>
+        <origin xyz="0 0 ${finger_length / 4}" rpy="0 0 0"/>      <!-- adjust offset/orientation if needed -->
+        <geometry>
+            <cylinder radius=".008" length="${finger_length / 2}"/>
+        </geometry>
+    </collision>
   </link>
   <joint name="ft_to_finger" type="fixed">
     <parent link="ft_link"/>
-    <origin xyz="0 0 ${ft_z}" rpy="0 0 0"/> <!-- adjust as needed -->
+    <origin xyz="0 0 ${ft_length}" rpy="0 0 0"/> <!-- adjust as needed -->
     <child link="finger_link"/>
   </joint>
@@ -71,5 +85,5 @@
   <joint name="finger_to_tip" type="fixed">
     <parent link="finger_link"/>
-    <origin xyz="0 0 ${finger_z}" rpy="0 0 0"/>
+    <origin xyz="0 0 ${finger_length}" rpy="0 0 0"/>
     <child link="finger_tip"/>
   </joint>

Commit message: too many problems with moveit, trying custom IK and Velocity control implemented

File: com_3d/urdf/irb120_with_finger.xacro (robot description, xacro)
@@ -8,7 +8,7 @@
   <xacro:property name="ft_mass" value="0.255"/>          <!-- kg (sensor) (from spec sheet) -->
   <xacro:property name="ft_cog_z" value="0.063"/>         <!-- meters in tool frame (from spec sheet)-->
-  <xacro:property name="ft_length" value="0.03"/>         <!-- FT sensor length -->
+  <xacro:property name="ft_length" value="0.08225"/>         <!-- FT sensor length -->
   <xacro:property name="finger_mass" value="0.066"/>      <!-- kg (finger) (from onshape) -->
-  <xacro:property name="finger_length" value="0.1143"/>   <!-- finger length (from onshape)-->
+  <xacro:property name="finger_length" value="0.110"/>   <!-- finger length (from onshape)-->
   <!-- Total offset from link_6 to finger tip will be ft_length + finger_length -->
   <!-- ====== FT sensor link mounted to link_6 ====== -->
@@ -20,5 +20,5 @@
     </inertial>
     <visual>
-      <origin xyz="0 0 ${ft_length/2}" rpy="0 0 0"/>
+      <origin xyz="0 0 ${ft_length / 2}" rpy="0 0 0"/>
       <geometry>
         <cylinder radius="0.025" length="${ft_length}"/>
@@ -30,7 +30,7 @@
     <!-- Basic cylinder collision geom -->
     <collision>
-        <origin xyz="0 0 ${ft_length / 4}" rpy="0 0 0"/>
+        <origin xyz="0 0 ${ft_length / 2}" rpy="0 0 0"/>
         <geometry>
-            <cylinder radius="0.025" length="${ft_length / 2}"/>
+            <cylinder radius="0.025" length="${ft_length / 2.5}"/>
         </geometry>
     </collision>
@@ -39,5 +39,5 @@
     <parent link="link_6"/>
     <!-- Adjust xyz/rpy to match your real mounting orientation -->
-    <origin xyz="0.001 0 0" rpy="0 1.5708 0"/>
+    <origin xyz="0 0 0" rpy="0 1.5708 0"/> <!-- Was 0.0001 0 0-->
     <child link="ft_link"/>
   </joint>

Commit message: Now recording untip motion as well. Added soda bottle experiment. Change to quat for apriltag orientation.

File: com_3d/urdf/irb120_with_finger.xacro (robot description, xacro)
@@ -13,4 +13,6 @@
   <xacro:property name="finger_length" value="0.110"/>   <!-- finger length (from onshape)-->
   <!-- Total offset from link_6 to finger tip will be ft_length + finger_length -->
+  <!-- Calibrated so that when finger_tip touches the table, FK reports z=-0.01199 in base_link -->
+  <xacro:property name="table_to_base_z" value="0.01199"/>  <!-- meters -->
   <!-- ====== FT sensor link mounted to link_6 ====== -->
   <link name="ft_link">
@@ -89,3 +91,10 @@
     <child link="finger_tip"/>
   </joint>
+  <link name='table'/>
+  <!-- Table is the parent (world-ish), base_link is lifted above it by table_to_base_z -->
+  <joint name="table_to_base_link" type="fixed">
+    <parent link="table"/>
+    <origin xyz="0 0 ${table_to_base_z}" rpy="0 0 0"/>
+    <child link="base_link"/>
+  </joint>
 </robot>

Commit message: a lot. Fixed pose motion, added objects and post-loop estimate and adaptive push height

File: com_3d/urdf/irb120_with_finger.xacro (robot description, xacro)
@@ -14,5 +14,5 @@
   <!-- Total offset from link_6 to finger tip will be ft_length + finger_length -->
   <!-- Calibrated so that when finger_tip touches the table, FK reports z=-0.01199 in base_link -->
-  <xacro:property name="table_to_base_z" value="0.01199"/>  <!-- meters -->
+  <xacro:property name="table_to_base_z" value="0.035"/>  <!-- was 0.01199 meters -->
   <!-- ====== FT sensor link mounted to link_6 ====== -->
   <link name="ft_link">
